Commit message: use materials defined in pal_urdf_utils for camera

File: urdf/camera/realsense_d405.urdf.xacro (robot description, xacro)
@@ -13,8 +13,10 @@
  -->
 <robot xmlns:xacro="http://ros.org/wiki/xacro">
+  <xacro:property name="realsense_materials_defined" value="true" />
   <xacro:include filename="$(find realsense2_description)/urdf/_d405.urdf.xacro"/>
   <xacro:include filename="$(find pal_urdf_utils)/urdf/camera/realsense_d405.gazebo.xacro" />
   <!-- Macro -->
   <xacro:macro name="realsense_d405" params="parent *origin name:=camera use_nominal_extrinsics:=false add_plug:=false use_mesh:=false">
+    <xacro:property name="add_plug" value="${add_plug}" />
     <xacro:sensor_d405 name="${name}" parent="${parent}" use_nominal_extrinsics="${use_nominal_extrinsics}">
       <xacro:insert_block name="origin" />

File: urdf/camera/realsense_d435.urdf.xacro (robot description, xacro)
@@ -13,4 +13,5 @@
  -->
 <robot xmlns:xacro="http://ros.org/wiki/xacro">
+  <xacro:property name="realsense_materials_defined" value="true" />
   <xacro:include filename="$(find realsense2_description)/urdf/_d435.urdf.xacro"/>
   <xacro:include filename="$(find pal_urdf_utils)/urdf/camera/realsense_d435.gazebo.xacro" />

File: urdf/camera/realsense_d435i.urdf.xacro (robot description, xacro)
@@ -13,4 +13,5 @@
  -->
 <robot xmlns:xacro="http://ros.org/wiki/xacro">
+  <xacro:property name="realsense_materials_defined" value="true" />
   <xacro:include filename="$(find realsense2_description)/urdf/_d435i.urdf.xacro"/>
   <xacro:include filename="$(find pal_urdf_utils)/urdf/camera/realsense_d435i.gazebo.xacro" />

File: urdf/camera/realsense_d455.urdf.xacro (robot description, xacro)
@@ -13,4 +13,5 @@
  -->
 <robot xmlns:xacro="http://ros.org/wiki/xacro">
+  <xacro:property name="realsense_materials_defined" value="true" />
   <xacro:include filename="$(find realsense2_description)/urdf/_d455.urdf.xacro"/>
   <xacro:include filename="$(find pal_urdf_utils)/urdf/camera/realsense_d455.gazebo.xacro" />

File: urdf/materials.urdf.xacro (robot description, xacro)
@@ -47,3 +47,9 @@
     <color rgba="0.29804 0.29804 0.29804 1"/>
   </material>
+  <material name="aluminum">
+    <color rgba="0.5 0.5 0.5 1"/>
+  </material>
+  <material name="plastic">
+    <color rgba="0.1 0.1 0.1 1"/>
+  </material>
 </robot>
