Commit message: add use_mesh and add_plug and set to False for d435i and d455

File: urdf/camera/realsense_d435i.urdf.xacro (robot description, xacro)
@@ -17,5 +17,5 @@
   <xacro:include filename="$(find pal_urdf_utils)/urdf/camera/realsense_d435i.gazebo.xacro" />
   <!-- Macro -->
-  <xacro:macro name="realsense_d435i" params="parent *origin name:=camera use_nominal_extrinsics:=false">
+  <xacro:macro name="realsense_d435i" params="parent *origin name:=camera use_nominal_extrinsics:=false add_plug:=false use_mesh:=false">
     <xacro:sensor_d435i name="${name}" parent="${parent}" use_nominal_extrinsics="${use_nominal_extrinsics}">
       <xacro:insert_block name="origin" />

File: urdf/camera/realsense_d455.urdf.xacro (robot description, xacro)
@@ -17,5 +17,5 @@
   <xacro:include filename="$(find pal_urdf_utils)/urdf/camera/realsense_d455.gazebo.xacro" />
   <!-- Macro -->
-  <xacro:macro name="realsense_d455" params="parent *origin name:=camera use_nominal_extrinsics:=false">
+  <xacro:macro name="realsense_d455" params="parent *origin name:=camera use_nominal_extrinsics:=false add_plug:=false use_mesh:=false">
     <xacro:sensor_d455 name="${name}" parent="${parent}" use_nominal_extrinsics="${use_nominal_extrinsics}">
       <xacro:insert_block name="origin" />
