Commit message: renamed to picoscan150core

File: urdf/laser/sick_picoscan150core_laser.gazebo.xacro (robot description, xacro)
@@ -13,10 +13,10 @@
  -->
 <robot xmlns:xacro="http://ros.org/wiki/xacro">
-  <xacro:macro name="sick_picoscan_laser_gazebo" params="name ros_topic update_rate min_angle max_angle">
-    <gazebo reference="${name}_link_1">
+  <xacro:macro name="sick_picoscan150core_laser_gazebo" params="name ros_topic update_rate min_angle max_angle">
+    <gazebo reference="${name}_link">
       <sensor name="${name}" type="gpu_lidar">
         <update_rate>${update_rate}</update_rate>
         <topic>${ros_topic}</topic>
-        <gz_frame_id>${name}_link_1</gz_frame_id>
+        <gz_frame_id>${name}_link</gz_frame_id>
         <visualize>true</visualize>
         <always_on>true</always_on>
@@ -49,5 +49,5 @@
             </ros>
             <output_type>sensor_msgs/LaserScan</output_type>
-            <frame_name>${name}_link_1</frame_name>
+            <frame_name>${name}_link</frame_name>
           </plugin>
         </xacro:if>
@@ -55,5 +55,5 @@
       <material>Gazebo/DarkGrey</material>
     </gazebo>
-    <gazebo reference="${name}_imu_link_1">
+    <gazebo reference="${name}_imu_link">
       <sensor name="${name}_imu_sensor" type="imu">
         <always_on>1</always_on>

File: urdf/laser/sick_picoscan_laser.urdf.xacro (robot description, xacro)
@@ -13,7 +13,7 @@
  -->
 <robot xmlns:xacro="http://ros.org/wiki/xacro">
-  <xacro:include filename="$(find pal_urdf_utils)/urdf/laser/sick_picoscan_laser.gazebo.xacro" />
-  <xacro:macro name="sick_picoscan_laser" params="name parent *origin ros_topic update_rate min_angle max_angle">
-    <link name="${name}_link_1" type="laser">
+  <xacro:include filename="$(find pal_urdf_utils)/urdf/laser/sick_picoscan150core_laser.gazebo.xacro" />
+  <xacro:macro name="sick_picoscan150core_laser" params="name parent *origin ros_topic update_rate min_angle max_angle">
+    <link name="${name}_link" type="laser">
       <inertial>
         <origin xyz="-0.02559000000 -0.00056000000 -0.05732000000" rpy="0 0 0"/>
@@ -24,5 +24,5 @@
         <origin xyz="0 0 0" rpy="1.57 0 1.57" />
         <geometry>
-          <!--<mesh filename="package://pal_urdf_utils/meshes/laser/sick_picoscan.stl" scale="0.001 0.001 0.001"/>-->
+          <!--<mesh filename="package://pal_urdf_utils/meshes/laser/sick_picoscan150core.stl" scale="0.001 0.001 0.001"/>-->
         </geometry>
         <material name="DarkGrey"/>
@@ -39,14 +39,14 @@
       <xacro:insert_block name="origin"/>
       <parent link="${parent}"/>
-      <child link="${name}_link_1"/>
+      <child link="${name}_link"/>
     </joint>
-    <link name="${name}_imu_link_1" type="imu"/>
+    <link name="${name}_imu_link" type="imu"/>
     <joint name="${name}_imu_joint" type="fixed">
-      <parent link="${name}_link_1"/>
-      <child link="${name}_imu_link_1"/>
-      <origin xyz="0.012 0.0185 0.0484" rpy="0 0 0"/>
+      <parent link="${name}_link"/>
+      <child link="${name}_imu_link"/>
+      <origin xyz="0.012 0.0185 0.0484" rpy="0 0 0"/>  <!-- position computed respect to the optical center of the laser z:0.0628 -->
     </joint>
     <!-- gazebo extensions -->
-    <xacro:sick_picoscan_laser_gazebo name="${name}" ros_topic="${ros_topic}" update_rate="${update_rate}" min_angle="${min_angle}" max_angle="${max_angle}"/>
+    <xacro:sick_picoscan150core_laser_gazebo name="${name}" ros_topic="${ros_topic}" update_rate="${update_rate}" min_angle="${min_angle}" max_angle="${max_angle}"/>
   </xacro:macro>
 </robot>
