Commit message: mesh visualization

File: urdf/laser/sick_picoscan_laser.urdf.xacro (robot description, xacro)
@@ -24,5 +24,5 @@
         <origin xyz="0 0 0" rpy="1.57 0 1.57" />
         <geometry>
-          <mesh filename="package://pal_urdf_utils/meshes/laser/sick_picoscan.stl" scale="0.001 0.001 0.001"/>
+          <!--<mesh filename="package://pal_urdf_utils/meshes/laser/sick_picoscan.stl" scale="0.001 0.001 0.001"/>-->
         </geometry>
         <material name="DarkGrey"/>

Commit message: added picoscan mesh

File: urdf/laser/sick_picoscan_laser.urdf.xacro (robot description, xacro)
@@ -24,5 +24,5 @@
         <origin xyz="0 0 0" rpy="1.57 0 1.57" />
         <geometry>
-          <!--<mesh filename="package://pal_urdf_utils/meshes/laser/sick_picoscan150core.stl" scale="0.001 0.001 0.001"/>-->
+          <mesh filename="package://pal_urdf_utils/meshes/laser/sick_picoscan150core.stl" scale="0.001 0.001 0.001"/>
         </geometry>
         <material name="DarkGrey"/>
