Commit message: added imu tracking link

File: urdf/laser/sick_picoscan150core_laser.urdf.xacro (robot description, xacro)
@@ -14,5 +14,9 @@
 <robot xmlns:xacro="http://ros.org/wiki/xacro">
   <xacro:include filename="$(find pal_urdf_utils)/urdf/laser/sick_picoscan150core_laser.gazebo.xacro" />
-  <xacro:macro name="sick_picoscan150core_laser" params="name parent *origin ros_topic update_rate min_angle max_angle">
+  <xacro:macro name="sick_picoscan150core_laser" params="name parent *origin ros_topic update_rate min_angle max_angle upsidedown:=false">
+  <xacro:property name="imu_R" value="0"/>
+  <xacro:if value="${upsidedown}">
+    <xacro:property name="imu_R" value="${180 * deg_to_rad}"/>
+  </xacro:if>
     <link name="${name}_link" type="laser">
       <inertial>
@@ -47,4 +51,10 @@
       <origin xyz="0.012 0.0185 0.0484" rpy="0 0 0"/>  <!-- position computed respect to the optical center of the laser z:0.0628 -->
     </joint>
+    <joint name="imu_tracking_joint" type="fixed">
+      <parent link="${name}_link"/>
+      <child link="imu_tracking_link"/>
+      <origin xyz="0.012 0.0185 0.0484" rpy="${imu_R} 0 0"/>
+    </joint>
+    <link name="imu_tracking_link"/>
     <!-- gazebo extensions -->
     <xacro:sick_picoscan150core_laser_gazebo name="${name}" ros_topic="${ros_topic}" update_rate="${update_rate}" min_angle="${min_angle}" max_angle="${max_angle}"/>

Commit message: update link and joint name

File: urdf/laser/sick_picoscan150core_laser.urdf.xacro (robot description, xacro)
@@ -51,10 +51,10 @@
       <origin xyz="0.012 0.0185 0.0484" rpy="0 0 0"/>  <!-- position computed respect to the optical center of the laser z:0.0628 -->
     </joint>
-    <joint name="imu_tracking_joint" type="fixed">
+    <joint name="${name}_imu_tracking_joint" type="fixed">
       <parent link="${name}_link"/>
-      <child link="imu_tracking_link"/>
+      <child link="${name}_imu_tracking_link"/>
       <origin xyz="0.012 0.0185 0.0484" rpy="${imu_R} 0 0"/>
     </joint>
-    <link name="imu_tracking_link"/>
+    <link name="${name}_imu_tracking_link"/>
     <!-- gazebo extensions -->
     <xacro:sick_picoscan150core_laser_gazebo name="${name}" ros_topic="${ros_topic}" update_rate="${update_rate}" min_angle="${min_angle}" max_angle="${max_angle}"/>
